File: PCB_Design/PCB_Design_PFE.kicad_pcb (KiCad board)
At the start: 4 copper layers, 62.9 x 42.5 mm, 64 parts, among them IC1 MAX86141ENP+, J1 Conn_01x02, U1 ADS1292RIPBS, U2 LSM6DSOX, U3 SHTC3, U4 TMP117AIDRVR, U5 STM32H7A3VITxQ, Y1 32,768 khz

Commit message: refactor: reorganisation claire (FreeRtos/, PCB_Design/, report/)
Parts:
- C28, C32, C33, C34, C35, C38, IC1, R9, U1, U4, U6: moved to B.Cu
- moved C33 49.4 mm to (122.4, 92.8), turned to 90 degrees
- moved C32 48.7 mm to (128.7, 99.9)
- moved U1 48.6 mm to (122.8, 98.6)
- moved U6 44.7 mm to (119.5, 87.6), turned to -90 degrees
- moved C30 41.6 mm to (104.2, 65.5)
- moved U2 41.6 mm to (100.9, 64.8)
- moved C31 41.6 mm to (100.4, 67.8)
- moved IC1 19.9 mm to (127.3, 85.5)
- moved C38 19.2 mm to (124.5, 85.2)
- moved C34 14.7 mm to (127.0, 82.9), turned to 90 degrees
- moved C35 14.7 mm to (128.5, 82.9), turned to 90 degrees
- moved R9 11.2 mm to (90.2, 67.6)
- moved U4 10.7 mm to (87.2, 66.5)
- moved C28 10.7 mm to (90.2, 66.2)
Routing:
- net GND: vias 1 -> 5
